Commit message: added gripper and FT to description

File: husky_custom_description/urdf/custom_description.urdf.xacro (robot description, xacro)
@@ -28,4 +28,31 @@
   <xacro:husky_robot />
   <!-- Insert Customizations Below -->
+  <xacro:include filename="$(find robotiq_s_model_visualization)/cfg/s-model_articulated_macro.xacro" />
+  <!-- Spawn and Join Gripper -->
+  <xacro:s-model_articulated prefix="" />
+  <joint name="gripper_base" type="fixed">
+    <parent link="ur5_arm_ee_link" />
+      <child link="palm" />
+      <origin xyz="0.11 0.0 0.0" rpy="0.0 -0.784 -1.57" />
+  </joint>
+  <!-- Sensor Mount and other custom parts -->
+  <link name="FT300_link">
+    <visual>
+      <geometry>
+        <cylinder length="0.06" radius="0.035"/>
+      </geometry>
+      <material name="black"/>
+    </visual>
+            <collision>
+                <geometry>
+                    <cylinder length="0.0475" radius="0.035"/>
+                </geometry>
+            </collision>
+       </link>
+      <joint name="FT300_joint" type="fixed">
+          <origin xyz="0.03 0 0" rpy="0 1.57 0" />
+          <parent link="ur5_arm_ee_link" />
+          <child link="FT300_link" />
+      </joint>
   <!-- Spawn the KAUST02 sensors mesh -->
   <link name="sensors_link">

Commit message: Working launch

File: husky_custom_description/urdf/custom_description.urdf.xacro (robot description, xacro)
@@ -22,6 +22,6 @@
 -->
 <robot name="husky" xmlns:xacro="http://ros.org/wiki/xacro">
-  <xacro:arg name="laser_enabled" default="$(optenv HUSKY_LMS1XX_ENABLED false)" />
-  <xacro:arg name="ur5_enabled" default="$(optenv HUSKY_UR5_ENABLED false)" />
+  <xacro:arg name="laser_enabled" default="false" />
+  <xacro:arg name="ur5_enabled" default="true" />
   <xacro:arg name="kinect_enabled" default="false" />
   <xacro:include filename="$(find husky_description)/urdf/husky.urdf.xacro" />
@@ -68,10 +68,3 @@
     <origin xyz="0.047 0.0 0.225" rpy="0.0 0.0 0.0" />
   </joint>
-  <link name="top_plate_link">
-  </link>
-  <joint name="top_joint" type="fixed">
-    <parent link="base_link" />
-    <child link="top_plate_link" />
-    <origin xyz="0.047 0.0 0.225" rpy="0.0 0.0 0.0" />
-  </joint>
 </robot>
